File: ogre/ogre.kicad_pcb (KiCad board)
At the start: 2 copper layers, 142 parts, among them U1 ProMicro

Commit message: v0
Parts:
- added SW1: SW_Push, Button_Switch_THT:SW_PUSH_6mm, F.Cu at (198.7, 98.3)
- added ogre-template: pcb-template, ogre:pcb-template, F.Cu at (35.2, 34.3)
- MX44: renamed from MX43; footprint Keebio:MX_PCB_100H -> Keebio:MX_PCB_225H
- MX45: renamed from MX44; footprint Keebio:MX_PCB_225H -> Keebio:MX_PCB_100H
- MX54: renamed from MX55; footprint Keebio:MX_PCB_225H -> Keebio:MX_PCB_100H
- MX55: renamed from MX56; footprint Keebio:MX_PCB_100H -> Keebio:MX_PCB_225H
- moved D56 338.0 mm to (355.1, 41.2), turned to 270 degrees
- moved D55 305.3 mm to (337.9, 97.9), turned to 270 degrees
- moved D69 301.3 mm to (317.6, 117.4), turned to 270 degrees
- moved D54 290.5 mm to (317.5, 98.6), turned to 270 degrees
- moved D68 289.7 mm to (298.5, 112.5), turned to 270 degrees
- moved D52 284.0 mm to (279.3, 91.5), turned to 270 degrees
- moved D42 284.0 mm to (336.4, 78.0), turned to 270 degrees
- moved D53 281.6 mm to (298.7, 93.5), turned to 270 degrees
- moved D14 281.5 mm to (336.7, 42.0), turned to 270 degrees
- moved D28 281.3 mm to (336.4, 59.0), turned to 270 degrees
- moved D2 280.4 mm to (70.0, 41.3), turned to 270 degrees
- moved D67 277.4 mm to (279.4, 110.2), turned to 270 degrees
- moved D26 276.9 mm to (298.4, 55.7), turned to 270 degrees
- moved D13 274.7 mm to (317.6, 41.3), turned to 270 degrees
- moved D12 273.0 mm to (298.3, 36.5), turned to 270 degrees
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- renumbered D49 to D43, D43 to D44, D44 to D45, D45 to D46, D46 to D47, D47 to D48, D48 to D49, D51 to D50, D52 to D51, D53 to D52, D54 to D53, D55 to D54, D56 to D55, D50 to D56, MX49 to MX43, MX45 to MX46, MX46 to MX47, MX47-Tab to MX48, MX48 to MX49, MX51 to MX50, MX52 to MX51, MX53 to MX52, MX54 to MX53, MX50 to MX56
Connections:
- MX10 pad 1: Col2 -> Col4
- MX12 pad 1: Col4 -> Col2
- MX13 pad 1: Col5 -> Col1
- MX14 pad 1: Col6 -> Col0
- MX22 pad 1: Col0 -> Col6
- MX23 pad 1: Col1 -> Col5
- MX24 pad 1: Col2 -> Col4
- MX26 pad 1: Col4 -> Col2
- MX27 pad 1: Col5 -> Col1
- MX28 pad 1: Col6 -> Col0
- MX36 pad 1: Col0 -> Col6
- MX37 pad 1: Col1 -> Col5
- MX38 pad 1: Col2 -> Col4
- MX40 pad 1: Col4 -> Col2
- MX41 pad 1: Col5 -> Col1
- MX42 pad 1: Col6 -> Col0
- MX50 pad 1: Col1 -> Col5
- MX51 pad 1: Col2 -> Col4
- MX53 pad 1: Col4 -> Col2
- MX54 pad 1: Col5 -> Col1
- MX55 pad 1: Col6 -> Col0
- MX56 pad 1: Col0 -> Col6
- MX64 pad 1: Col0 -> Col6
- MX65 pad 1: Col1 -> Col5
- MX66 pad 1: Col2 -> Col4
- MX68 pad 1: Col4 -> Col2
- MX69 pad 1: Col5 -> Col1
- MX70 pad 1: Col6 -> Col0
- MX8 pad 1: Col0 -> Col6
- MX9 pad 1: Col1 -> Col5
- U1 pad 10: Row6 -> Col1
- U1 pad 11: Row7 -> Col2
- U1 pad 12: Row8 -> Col3
- U1 pad 16: Col3 -> Row9
- U1 pad 17: Col2 -> Row8
- U1 pad 18: Col1 -> Row7
- U1 pad 19: Col0 -> Row6
- U1 pad 20: Row9 -> Row5
- U1 pad 9: Row5 -> Col0
Routing:
- net Col6: track 0.00 -> 585.8 mm
- net Col0: track 0.00 -> 526.8 mm, vias 0 -> 3
- net Col2: track 0.00 -> 437.9 mm, vias 0 -> 6
- net Col1: track 0.00 -> 431.8 mm, vias 0 -> 4
- net Col3: track 0.00 -> 361.5 mm, vias 0 -> 7
- net Col4: track 0.00 -> 353.4 mm, vias 0 -> 6
- net Col5: track 0.00 -> 338.6 mm, vias 0 -> 4
- net Row3: track 0.00 -> 298.6 mm
- net Row8: track 0.00 -> 262.1 mm
- net Row4: track 0.00 -> 234.4 mm
- net Row9: track 0.00 -> 223.6 mm
- net Row2: track 0.00 -> 192.6 mm
- net Row1: track 0.00 -> 172.5 mm
- net Row7: track 0.00 -> 165.1 mm
- net Row0: track 0.00 -> 155.7 mm
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Other:
- net class Default: clearance 0.2 -> 0.5; trace_width 0.25 -> 0.5; via_dia 0.8 -> 0.6; via_drill 0.4 -> 0.3
- rule pad_to_mask_clearance: 0.051 -> 0.075
- rule solder_mask_min_width: 0.25 -> 0.15
- rule trace_clearance: 0.2 -> 0.5
- rule trace_min: 0.2 -> 0.5
- rule via_min_size: 0.4 -> 0.6

Commit message: placed
Parts:
- removed ogre-plate: ogre-plate, ogre.temp:ogre-plate
- moved D28 1.34 mm to (336.3, 60.3)
- moved D14 0.79 mm to (336.4, 41.2)
- moved MX69 0.57 mm to (325.2, 116.1)
- moved MX10 0.56 mm to (268.1, 35.1)
- moved D20 0.55 mm to (146.0, 57.9)
- moved MX50 0.51 mm to (249.1, 94.6)
- moved MX11 0.51 mm to (287.2, 32.7)
- moved MX52 0.51 mm to (287.2, 89.9)
- moved MX53 0.51 mm to (306.2, 92.3)
- moved MX37 0.51 mm to (249.1, 75.6)
- moved MX38 0.51 mm to (268.1, 73.2)
- moved MX67 0.51 mm to (287.2, 108.9)
- moved MX23 0.51 mm to (249.1, 56.5)
- moved MX24 0.51 mm to (268.1, 54.2)
- moved MX42 0.51 mm to (351.4, 78.0)
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Routing:
- net Col6: track 585.8 -> 0.00 mm
- net Col0: track 526.8 -> 0.00 mm, vias 3 -> 0
- net Col2: track 437.9 -> 0.00 mm, vias 6 -> 0
- net Col1: track 431.8 -> 0.00 mm, vias 4 -> 0
- net Col3: track 361.5 -> 0.00 mm, vias 7 -> 0
- net Col4: track 353.4 -> 0.00 mm, vias 6 -> 0
- net Col5: track 338.6 -> 0.00 mm, vias 4 -> 0
- net Row3: track 298.6 -> 0.00 mm
- net Row8: track 262.1 -> 0.00 mm
- net Row4: track 234.4 -> 0.00 mm
- net Row9: track 223.6 -> 0.00 mm
- net Row2: track 192.6 -> 0.00 mm
- net Row1: track 172.5 -> 0.00 mm
- net Row7: track 165.1 -> 0.00 mm
- net Row0: track 155.7 -> 0.00 mm
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
Commit message: start flipping diodes
Parts:
- added MX71: MX-NoLED, Keebio:MX_PCB_125H, F.Cu at (346.7, 78.0)
- added MX72: MX-NoLED, Keebio:MX_PCB_125H, F.Cu at (346.7, 97.0)
- added MX73: MX-NoLED, Keebio:MX_PCB_125H, F.Cu at (327.7, 116.1)
- added MX74: MX-NoLED, Keebio:MX_PCB_125H, F.Cu at (75.7, 116.3)
- added REF**: pcb-outline, ogre:pcb-outline, F.Cu at (0.69, 156.9)
- added SW2: SW_Push, Button_Switch_THT:SW_PUSH_6mm, F.Cu at (166.5, 87.4)
- added SW3: SW_Push, Button_Switch_THT:SW_PUSH_6mm, F.Cu at (229.4, 87.4)
- added U2: ProMicro, Keebio:ArduinoProMicro, F.Cu at (173.4, 45.2)
- added U3: ProMicro, Keebio:ArduinoProMicro, F.Cu at (230.0, 45.1)
- D1, D10, D11, D12, D13, D14, D2, D3, D4, D43, D5, D56, D6, D7, D8, D9: moved to B.Cu
- moved D7 10.8 mm to (173.2, 45.9), turned to 0 degrees
- moved D8 10.5 mm to (230.1, 45.7), turned to 0 degrees
- moved D21 10.5 mm to (173.2, 64.6), turned to 0 degrees
- moved D22 10.4 mm to (229.7, 65.1), turned to 0 degrees
- moved D58 3.51 mm to (66.3, 117.3)
- moved D69 0.62 mm to (317.0, 117.3)
Routing:
- net Net-(D7-Pad2): track 4.55 -> 0.00 mm
- net Net-(D21-Pad2): track 4.42 -> 0.00 mm
- net Net-(D8-Pad2): track 4.00 -> 0.00 mm
- net Net-(D22-Pad2): track 3.99 -> 0.00 mm
Other:
- board outline added: 346.4 x 129.7 mm

Commit message: grids done
Parts:
- removed REF**: pcb-outline, ogre:pcb-outline
- D15, D16, D17, D18, D19, D20, D21, D22, D23, D24, D25, D26, D27, D28, D29, D30, D31, D32, D33, D34, D35, D36, D37, D38, D39, D40, D41, D42, D44, D45, D46, D47, D48, D49, D50, D51, D52, D53, D54, D55, D57, D58, D59, D60, D61, D62, D63, D64, D65, D66, D67, D68, D69, D70, SW1, SW2, SW3: moved to B.Cu
- moved ogre-template 127.3 mm to (0.69, 156.9)
- moved SW3 8.24 mm to (237.6, 87.0), turned to 180 degrees
- moved SW1 6.40 mm to (204.8, 99.9), turned to 180 degrees
- moved D8 5.49 mm to (226.1, 41.9), turned to 270 degrees
- moved D22 5.40 mm to (226.0, 61.1), turned to 270 degrees
- moved D7 5.31 mm to (169.5, 42.1), turned to 270 degrees
- moved D21 5.22 mm to (169.3, 61.1), turned to 270 degrees
- moved SW2 4.29 mm to (165.7, 91.6)
- moved D65 1.95 mm to (226.3, 104.9)
- moved D62 1.21 mm to (179.6, 101.2)
Routing:
- net Col6: track 0.00 -> 490.0 mm
- net Col5: track 0.00 -> 198.7 mm
- net Col0: track 0.00 -> 189.1 mm
- net Row3: track 0.00 -> 183.6 mm
- net Col4: track 0.00 -> 183.0 mm
- net Row8: track 0.00 -> 173.0 mm, vias 0 -> 1
- net Row4: track 0.00 -> 171.7 mm
- net Col1: track 0.00 -> 166.0 mm
- net Col2: track 0.00 -> 161.5 mm
- net Col3: track 0.00 -> 160.4 mm
- net Row0: track 0.00 -> 159.5 mm, vias 0 -> 3
- net Row9: track 0.00 -> 154.3 mm
- net Row1: track 0.00 -> 134.2 mm
- net Row2: track 0.00 -> 132.1 mm
- net Row7: track 0.00 -> 121.6 mm
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Other:
- board outline removed

Commit message: start on pro-micros
Parts:
- moved D23 14.3 mm to (255.6, 57.4)
- moved D9 13.7 mm to (255.0, 39.1)
Routing:
- net Row5: track 102.0 -> 251.9 mm, vias 0 -> 2
- net Row6: track 100.8 -> 184.0 mm
- net Row1: track 134.2 -> 199.2 mm
- net Row2: track 132.1 -> 190.2 mm
- net Row7: track 121.6 -> 178.4 mm
- net Col0: track 189.1 -> 239.2 mm
- net Row3: track 183.6 -> 231.7 mm
- net Row8: track 173.0 -> 221.0 mm
- net Col1: track 166.0 -> 209.4 mm
- net Col4: track 183.0 -> 222.3 mm
- net Row4: track 171.7 -> 210.7 mm
- net Row9: track 154.3 -> 192.9 mm
- net Col5: track 198.7 -> 230.6 mm
- net Col2: track 161.5 -> 185.9 mm
- net Col6: track 490.0 -> 469.1 mm
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
Commit message: wip
Parts:
- removed SW1: SW_Push, Button_Switch_THT:SW_PUSH_6mm
- removed U1: ProMicro, Keebio:ArduinoProMicro
- removed ogre-template: pcb-template, ogre:pcb-template
- moved U2 17.5 mm to (190.2, 40.6)
- moved U3 17.5 mm to (213.1, 40.8)
Routing:
- net Col6: track 469.1 -> 1.27 mm
- net Col0: track 239.2 -> 10.9 mm
- net Row5: track 251.9 -> 25.9 mm
- net Col5: track 230.6 -> 11.6 mm
- net Row3: track 231.7 -> 19.4 mm
- net Col4: track 222.3 -> 14.3 mm
- net Row8: track 221.0 -> 18.4 mm
- net Col1: track 209.4 -> 8.66 mm
- net Row4: track 210.7 -> 16.7 mm
- net Row9: track 192.9 -> 0.00 mm
- net Col2: track 185.9 -> 5.37 mm
- net Row1: track 199.2 -> 24.3 mm
- net Row2: track 190.2 -> 21.9 mm
- net Col3: track 168.2 -> 2.10 mm
- net Row6: track 184.0 -> 24.6 mm
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Other:
- net class Default: clearance 0.5 -> 0.2; trace_width 0.5 -> 0.25; via_drill 0.3 -> 0.4
- rule trace_clearance: 0.5 -> 0.2
- rule trace_min: 0.5 -> 0.2
- rule via_min_size: 0.6 -> 0.4

Commit message: right half almost done
Parts:
- added ogre4-cut: ogre4-cut, ogre:ogre4-cut, F.Cu at (-23.2, 0.00)
- added ogre4-ink: ogre4-ink, ogre:ogre4-ink, F.Cu at (-23.2, 0.00)
- moved SW2 79.3 mm to (188.1, 15.5)
- moved SW3 78.1 mm to (213.7, 12.7)
- moved D23 13.8 mm to (241.8, 57.9)
- moved D9 13.5 mm to (241.5, 38.9)
- moved D63 7.61 mm to (192.0, 117.2)
- moved D7 5.42 mm to (165.3, 38.6)
- moved D21 4.98 mm to (165.6, 57.8)
- moved D8 4.54 mm to (222.8, 38.9)
- moved D22 4.38 mm to (222.9, 58.0)
- moved U2 4.33 mm to (192.2, 44.5)
- moved U3 4.02 mm to (211.3, 44.5)
Connections:
- U2 pad 1: Net-(U2-Pad1) -> Row0
- U2 pad 10: Col1 -> Row2
- U2 pad 11: Col2 -> Row3
- U2 pad 12: Col3 -> Row4
- U2 pad 13: Col6 -> Net-(U2-Pad13)
- U2 pad 14: Col5 -> Col6
- U2 pad 15: Col4 -> Col5
- U2 pad 16: Row9 -> Col4
- U2 pad 17: Row8 -> Col3
- U2 pad 18: Row7 -> Col2
- U2 pad 19: Row6 -> Col1
- U2 pad 2: Net-(U2-Pad2) -> Row1
- U2 pad 20: Row5 -> Col0
- U2 pad 5: SDA -> Net-(U2-Pad5)
- U2 pad 6: SCL -> Net-(U2-Pad6)
- U2 pad 8: Net-(U2-Pad8) -> Row0
- U2 pad 9: Col0 -> Row1
- U3 pad 1: Net-(U3-Pad1) -> Row0
- U3 pad 10: Col1 -> Row7
- U3 pad 11: Col2 -> Row8
- U3 pad 12: Col3 -> Row9
- U3 pad 13: Col6 -> Net-(U3-Pad13)
- U3 pad 14: Col5 -> Col6
- U3 pad 15: Col4 -> Col5
- U3 pad 16: Row4 -> Col4
- U3 pad 17: Row3 -> Col3
- U3 pad 18: Row2 -> Col2
- U3 pad 19: Row1 -> Col1
- U3 pad 2: Net-(U3-Pad2) -> Row1
- U3 pad 20: Row0 -> Col0
- U3 pad 5: SDA -> Row2
- U3 pad 6: SCL -> Row3
- U3 pad 7: Net-(U3-Pad7) -> Row4
- U3 pad 8: Net-(U3-Pad8) -> Row5
- U3 pad 9: Col0 -> Row6
Routing:
- net Col6: track 1.27 -> 565.8 mm, vias 0 -> 1
- net Col0: track 10.9 -> 324.6 mm
- net Row3: track 19.4 -> 328.3 mm, vias 0 -> 1
- net Col1: track 8.66 -> 273.8 mm, vias 0 -> 1
- net Row4: track 16.7 -> 269.9 mm, vias 0 -> 1
- net Row1: track 24.3 -> 276.5 mm, vias 0 -> 1
- net Col2: track 5.37 -> 250.6 mm, vias 0 -> 1
- net Row2: track 21.9 -> 261.0 mm, vias 0 -> 1
- net Col3: track 2.10 -> 230.2 mm, vias 0 -> 1
- net Col5: track 11.6 -> 233.5 mm
- net Col4: track 14.3 -> 234.3 mm
- net Row8: track 18.4 -> 235.4 mm, vias 1 -> 0
- net Row9: track 0.00 -> 214.9 mm
- net Row0: track 27.4 -> 167.2 mm, vias 1 -> 0
- net Row7: track 22.1 -> 157.4 mm
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Other:
- board outline added: 351.9 x 129.5 mm

Commit message: wip
Parts:
- ogre4-cut: value ogre4-cut -> ogre4-cut-2; footprint ogre:ogre4-cut -> ogre:ogre4-cut-2
- moved SW3 65.4 mm to (214.8, 78.1)
- moved SW2 62.6 mm to (193.9, 77.8), turned to 180 degrees
Routing:
- net Col0: track 324.6 -> 600.5 mm, vias 0 -> 5
- net Col1: track 273.8 -> 471.7 mm, vias 1 -> 7
- net Col2: track 250.6 -> 448.4 mm, vias 1 -> 6
- net Col4: track 234.3 -> 431.8 mm, vias 0 -> 2
- net Col3: track 230.2 -> 391.3 mm, vias 1 -> 6
- net Col5: track 233.5 -> 386.0 mm, vias 0 -> 3
- net GND: track 0.00 -> 140.1 mm, vias 0 -> 1
- net Col6: track 565.8 -> 659.1 mm, vias 1 -> 4
- net Row2: track 261.0 -> 327.7 mm, vias 1 -> 4
- net Row3: track 328.3 -> 391.3 mm, vias 1 -> 3
- net Row4: track 269.9 -> 326.6 mm, vias 1 -> 2
- net RSTR: track 0.00 -> 54.6 mm, vias 0 -> 1
- net RSTL: track 0.00 -> 52.7 mm
- net Row1: track 276.5 -> 308.9 mm, vias 1 -> 5
- net Row0: track 167.2 -> 192.7 mm, vias 0 -> 1
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Other:
- board size 351.9 x 129.5 mm -> 351.9 x 130.4 mm
