File: ogre/ogre.kicad_pcb (KiCad board)
At the start: 2 copper layers, 351.9 x 130.4 mm, 150 parts, among them SW2 SW_Push, SW3 SW_Push, U2 ProMicro, U3 ProMicro

Commit message: retrace
Parts:
- added U21: TRRS, ogre.temp:PJ-3200B-4A, F.Cu at (200.9, 83.0)
- added U31: TRRS, ogre.temp:PJ-3200B-4A, F.Cu at (202.7, 83.0)
- MX21: footprint Keebio:MX_PCB_100H -> Keebio-Parts:MX_PCB_100H
- moved D44 36.1 mm to (64.4, 96.9)
- moved SW2 17.3 mm to (181.5, 90.0), turned to 330 degrees
- moved D43 16.5 mm to (48.3, 41.1)
- moved SW3 16.2 mm to (221.0, 93.1), turned to 30 degrees
- moved D57 1.93 mm to (48.1, 117.7)
- moved D69 1.14 mm to (318.1, 117.5)
Connections:
- U2 pad 1: Row0 -> SCL2
- U2 pad 2: Row1 -> SDA2
Routing:
- net (no net): track 0.00 -> 84.5 mm, vias 0 -> 1
- net GND: track 140.1 -> 87.4 mm, vias 1 -> 0
- net Net-(D42-Pad2): track 11.9 -> 21.8 mm
- net Col2: track 448.4 -> 440.5 mm
- net Col3: track 391.3 -> 386.3 mm
- net Row0: track 192.7 -> 197.6 mm
- net Col5: track 386.0 -> 382.2 mm
- net Col4: track 431.8 -> 428.0 mm
- net Row8: track 244.4 -> 248.0 mm
- net Col0: track 600.5 -> 603.5 mm
- net Col6: track 659.1 -> 660.7 mm
- net Net-(D36-Pad2): track 3.85 -> 5.23 mm
- net Net-(D14-Pad2): track 5.29 -> 4.14 mm
- net Net-(D12-Pad2): track 5.13 -> 4.09 mm
- net Net-(D9-Pad2): track 4.82 -> 3.79 mm
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
Commit message: rows and columns done
Parts:
- SW2, SW3: moved to F.Cu
- U21, U31: footprint ogre.temp:PJ-3200B-4A -> Keebio:TRRS-PJ-320A
- moved SW3 15.5 mm to (208.9, 83.4), turned to 0 degrees
- moved SW2 9.14 mm to (188.0, 83.5), turned to 0 degrees
- moved U21 6.78 mm to (198.8, 76.5), turned to 270 degrees
- moved U31 6.71 mm to (204.7, 76.6), turned to 90 degrees
- moved MX15 0.09 mm to (54.4, 59.0)
Routing:
- net Col0: track 603.5 -> 178.6 mm, vias 5 -> 0
- net Col6: track 660.7 -> 344.9 mm, vias 4 -> 0
- net Col1: track 472.6 -> 157.4 mm, vias 7 -> 0
- net Col2: track 440.5 -> 153.3 mm, vias 6 -> 0
- net Col4: track 428.0 -> 178.1 mm, vias 2 -> 0
- net Col3: track 386.3 -> 152.8 mm, vias 6 -> 0
- net Row3: track 391.3 -> 162.2 mm, vias 3 -> 2
- net Row2: track 326.7 -> 129.6 mm, vias 5 -> 0
- net Col5: track 382.2 -> 195.2 mm, vias 3 -> 1
- net Row1: track 308.8 -> 127.3 mm, vias 5 -> 0
- net Row4: track 327.2 -> 191.3 mm, vias 2 -> 3
- net GND: track 87.4 -> 0.00 mm
- net (no net): track 84.5 -> 0.00 mm, vias 1 -> 0
- net Row0: track 197.6 -> 121.1 mm, vias 1 -> 0
- net Row9: track 223.0 -> 164.3 mm, vias 2 -> 1
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
Commit message: only a few left
Routing:
- net Col0: track 178.6 -> 1023.1 mm, vias 0 -> 3
- net Col3: track 152.8 -> 520.6 mm, vias 0 -> 4
- net Col1: track 157.4 -> 459.4 mm, vias 0 -> 3
- net Col2: track 153.3 -> 410.8 mm, vias 0 -> 4
- net Col6: track 344.9 -> 572.3 mm, vias 0 -> 2
- net Col5: track 195.2 -> 374.2 mm, vias 1 -> 3
- net Col4: track 178.1 -> 349.6 mm, vias 0 -> 3
- net Row3: track 162.2 -> 323.7 mm, vias 2 -> 4
- net Row1: track 127.3 -> 248.8 mm, vias 0 -> 3
- net Row2: track 129.6 -> 248.1 mm, vias 0 -> 2
- net Row4: track 191.3 -> 306.8 mm, vias 3 -> 5
- net Row0: track 121.1 -> 235.6 mm, vias 0 -> 3
- net VCC: track 0.00 -> 91.4 mm, vias 0 -> 2
- net Row8: track 190.0 -> 270.0 mm, vias 1 -> 2
- net Row9: track 164.3 -> 232.2 mm, vias 1 -> 4
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
Commit message: done
Parts:
- removed ogre4-ink: ogre4-ink, ogre:ogre4-ink
Routing:
- net GND: track 37.4 -> 157.2 mm, vias 1 -> 2
- net RSTL: track 6.50 -> 77.6 mm, vias 0 -> 3
- net Row5: track 166.8 -> 169.0 mm
